File: hardware/pcb/debug-helper/rev-a/dutchmate_debug_helper.kicad_sch (KiCad schematic)
At the start: 41 parts, among them J1 Conn_02x08_Odd_Even, U1 SN74LV4T125, U2 TXU0202DCUR, U4 TPD6E05U06RVZ, U5 TXU0104PWR, U6 TPD4E05U06DQA, U7 SN74LVC2G06DBV, U8 SN74LVC2G06DBV

Commit message: Finalize Rev-A KiCad source corrections
Signed-off-by: Nahit Pawar <nahitpawar@gmail.com>
Parts:
- added C16: 100nF, Capacitor_SMD:C_0603_1608Metric, symbol Device:C_Small
- added R14, R15, R16, R17: 10K, Resistor_SMD:R_0603_1608Metric, symbol Device:R_Small
- added U3: TMUX2819DSGR, Package_SON:Texas_DSG0008A_WSON-8-1EP_2x2mm_P0.5mm_EP0.9x1.6mm, symbol dutchmate:TMUX2819
- A1: value RaspberryPi_Pico -> Raspberry Pi Pico 2
- R1, R2, R3, R4: value 100K -> 4.7K
- R12, R5: value 10K -> 4.7K
- R13: value 47K -> 10K
- R6, R7, R8, R9: value 47K -> 4.7K
- RN3, RN4: value 181R -> 180R
Connections:
- net +3.3V: now also C16.1, U3.3 (EN), U3.8 (VDD)
- net DBG_CTRL_DATA0: now also R14.1
- net DBG_CTRL_DATA1: now also R15.1
- net DBG_CTRL_DATA2: now also R16.1
- net DBG_CTRL_DATA3: now also R17.1
- net DUT_VIO: now also U3.1 (SA); no longer R10.1
- net GND: now also C16.2, R14.2, R15.2, R16.2, R17.2, U3.2 (NC), U3.4 (GND), U3.7 (SEL), U3.9 (GND); no longer A1.33 (AGND), C7.2, R11.2
- net DBG_CTRL_OE3_N: now reaches R8.2, U1.13, U8.6 (1Y)
- net DBG_CTRL_OE0_N: now reaches R7.2, U1.1, U7.4 (2Y)
- net DBG_CTRL_OE1_N: now reaches R6.2, U1.4, U7.6 (1Y)
- net DBG_CTRL_OE2_N: now reaches R9.2, U1.10, U8.4 (2Y)
- new net: R10.1, U3.6 (D)
- new net GNDA: A1.33 (AGND), C7.2, R11.2
- no-connect marks 0 -> 15
Other:
- moved on the sheet: A1, C1, C11, C12, C13, C14, C15, C2, C5, C6, C7, C8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
